File: epopee du poulet/Kicad/epopee_du_poulet/epopee_du_poulet.kicad_sch (KiCad schematic)
At the start: 8 parts, among them SW2 SW_Push_Dual, U1 ATmega328-P, U2 93CxxC, U3 DS1307+, Y1 Crystal

Commit message: coucou toi
Parts:
- removed R1: R, symbol Device:R
- removed SW2: SW_Push_Dual, symbol Switch:SW_Push_Dual

Commit message: ajout du kicad
Parts:
- added C2, C4: 100nF, Capacitor_SMD:C_0805_2012Metric_Pad1.18x1.45mm_HandSolder, symbol Device:C
- added J2: CP2102 PINS, Connector_PinSocket_2.54mm:PinSocket_1x06_P2.54mm_Vertical, symbol Connector:Conn_01x06_Socket
- added R1: 10kOhm, Resistor_THT:R_Axial_DIN0204_L3.6mm_D1.6mm_P2.54mm_Vertical, symbol Device:R
- added SW1: ResetButton, Button_Switch_THT:SW_PUSH_6mm, symbol Switch:SW_Push_Dual
- BT1: value Battery_Cell -> CR2025; footprint (none) -> Battery:Battery_Panasonic_CR2032-HFN_Horizontal_CircularHoles
- C1: value C -> 100nF; footprint (none) -> Capacitor_SMD:C_0805_2012Metric_Pad1.18x1.45mm_HandSolder
- U1: value ATmega328-P -> ATmega328P
- U2: value 93CxxC -> 93C06; footprint (none) -> Package_DIP:DIP-8_W7.62mm
- U3: value DS1307+ -> DS1307
- Y1: value Crystal -> 32kHz; footprint (none) -> Crystal:Crystal_Round_D3.0mm_Vertical
Connections:
- net VCC is gone; now on net +5V: C1.2, U2.8 (VCC)
- net +5V: now also U3.8 (VCC), C2.2, J2.1 (Pin_1), R1.2
- net GND: now also BT1.2 (-), U1.22 (GND), U1.8 (GND), U3.4 (GND), C2.1, J2.2 (Pin_2), SW1.2
- net at U1.1 (~{RESET}/PC6): now also C4.1, R1.1, SW1.1
- net rx: no longer names the net of U1.2 (PD0)
- net rx: now also J2.3 (Pin_3)
- net tx: no longer names the net of U1.3 (PD1)
- net tx: now also J2.4 (Pin_4)
- new net: C4.2, J2.5 (Pin_5)
Other:
- moved on the sheet: BT1, U3, Y1
