File: epopee du poulet/Kicad/epopee_du_poulet/epopee_du_poulet.kicad_pcb (KiCad board)
At the start: 2 copper layers, 11 parts, among them J2 CP2102 PINS, SW1 ResetButton, U1 ATmega328P, U2 93C06, U3 DS1307, Y1 32kHz

Commit message: derniere version du pcb
Routing:
- net Net-(U1-PD7): track 57.0 -> 46.0 mm
- net Net-(U1-~{RESET}/PC6): track 31.1 -> 34.8 mm
- net Net-(U1-PC4): track 94.0 -> 91.7 mm
- net +5V: track 129.3 -> 131.5 mm
- net Net-(U1-PB2): track 28.7 -> 29.9 mm
- net GND: track 160.9 -> 161.5 mm
